File: kicad-files/Sync-Ope-proto.sch (KiCad schematic (older format))
At the start: 31 parts, among them J1 VIDEO_INPUT, J2 VIDEO_SEND, J3 VIDEO_RETURN, J4 VIDEO_OUTPUT, U1 4069, U2 AD8072, U3 LM1881, U4 LT1251

Commit message: wip - updating schematic, not finished
Parts:
- removed C1: 100nF, symbol C
- removed D1, D2: D, symbol D
- removed R1: 75, symbol R
- removed R2, R9: 220, symbol R
- removed R3, R4: 1.5k, symbol R
- removed R5: 10k, symbol R
- removed R6: 100, symbol R
- removed R8: 6.8k, symbol R
- removed RV1: POT, symbol POT
- removed U1: 4069, symbol 4069
- removed U2: AD8072, symbol AD8072
- added C? (x2): 100n, symbol C
- added J?: CV WET/DRY, symbol Audio-Jack-2
- added Q? (x2): 2N2219, TO_SOT_Packages_THT:TO-39-3, symbol 2N2219
- added Q?: 2N7000, TO_SOT_Packages_THT:TO-92_Molded_Narrow, symbol 2N7000
- added Q?: 2N3904, TO_SOT_Packages_THT:TO-92_Molded_Narrow, symbol 2N3904
- added R? (x3): 10k, symbol R
- added R?: 4.7k, symbol R
- added R? (x4): r, symbol R
- added R?: 220, symbol R
- added R? (x6): 100k, symbol R
- added R? (x2): 75, symbol R
- added R? (x2): 1k, symbol R
- added R?: 1.4k, symbol R
- added RV?: WET/DRY, symbol POT
- added U? (x3): LM6172, symbol LM6172
- added U?: 4053, symbol 4053
Connections:
- net labels added: FADER_LEVEL, VIDEO_TO_BLACK_RESTORE
- net labels removed: VDD, VSS
- wire segments 94 -> 119
- no-connect marks 11 -> 7
Other:
- note added: "Input buffer and send"
- note added: "Transistor AND gate"
- note added: "Video Fader"
- note added: "dry/wet control"
- note removed: "CV Video Fader"
- note removed: "Dual Video Amplifier"
- note removed: "Hex-inverter AND gate"
- moved on the sheet: J2, J3, J4, R10, R11, R12, R13, R14, R15, R16, R17, U4
