File: kicad-files/Sync-Ope-proto.sch (KiCad schematic (older format))
At the start: 47 parts, among them J1 VIDEO_INPUT, J2 euro_power, J3 VIDEO_SEND, J4 VIDEO_RETURN, J5 CV_IN, J6 VIDEO_OUTPUT, U1 AD8072, U2 LM1881, U3 L7805, U4 L7905, U5 LT1251, U6 CD4053BE

Commit message: updating schematic and pcb for 0.1proto
Parts:
- removed R3: 100, Resistor_THT:R_Axial_DIN0204_L3.6mm_D1.6mm_P5.08mm_Horizontal, symbol Sync-Ope-proto:R
- added C12, C13: 200u, Capacitor_THT:CP_Radial_D5.0mm_P2.50mm, symbol Device:CP_Small
- added D4, D5: 1n4007, Diode_THT:D_DO-35_SOD27_P7.62mm_Horizontal, symbol Device:D
- added D6: zener_1.8v, Diode_THT:D_DO-35_SOD27_P7.62mm_Horizontal, symbol Device:D_Zener
- added D7: schottky, Diode_THT:D_DO-35_SOD27_P7.62mm_Horizontal, symbol Device:D_Schottky
- added J7: AC_POWER, Connector_BarrelJack:BarrelJack_Horizontal, symbol Connector:Barrel_Jack
- added J8: diy_power_header, Connector_PinHeader_2.54mm:PinHeader_1x03_P2.54mm_Vertical, symbol Connector:Conn_01x03_Female
- added R3: 220, Resistor_THT:R_Axial_DIN0204_L3.6mm_D1.6mm_P5.08mm_Horizontal, symbol Device:R
- C3, C4, C5: symbol Sync-Ope-proto:C -> Sync-Ope-proto-rescue:C-Sync-Ope-proto
- J1, J6: symbol Sync-Ope-proto:Conn_Rca -> Sync-Ope-proto-rescue:Conn_Rca-Sync-Ope-proto
- R1, R11, R15, R17, R18, R19, R20, R4, R5, R6, R8, R9: symbol Sync-Ope-proto:R -> Sync-Ope-proto-rescue:R-Sync-Ope-proto
- R12: value 100k -> 470k; symbol Sync-Ope-proto:R -> Sync-Ope-proto-rescue:R-Sync-Ope-proto
- R13: value 100 -> 75; symbol Sync-Ope-proto:R -> Sync-Ope-proto-rescue:R-Sync-Ope-proto
- RV1: symbol Sync-Ope-proto:POT -> Sync-Ope-proto-rescue:POT-Sync-Ope-proto
- U1: symbol Sync-Ope-proto:AD8072 -> Sync-Ope-proto-rescue:AD8072-Sync-Ope-proto
- U2: symbol Sync-Ope-proto:LM1881 -> Sync-Ope-proto-rescue:LM1881-Sync-Ope-proto
- U5: symbol Sync-Ope-proto:LT1251 -> Sync-Ope-proto-rescue:LT1251-Sync-Ope-proto
Connections:
- wire segments 195 -> 214

Commit message: update a trace for proto0.1 order
Parts:
- C3, C4, C5: symbol Sync-Ope-proto-rescue:C-Sync-Ope-proto -> Sync-Ope-proto-rescue:C-Sync-Ope-proto-Sync-Ope-proto-rescue
- J1, J6: symbol Sync-Ope-proto-rescue:Conn_Rca-Sync-Ope-proto -> Sync-Ope-proto-rescue:Conn_Rca-Sync-Ope-proto-Sync-Ope-proto-rescue
- R1, R11, R12, R13, R15, R17, R18, R19, R20, R4, R5, R6, R8, R9: symbol Sync-Ope-proto-rescue:R-Sync-Ope-proto -> Sync-Ope-proto-rescue:R-Sync-Ope-proto-Sync-Ope-proto-rescue
- RV1: symbol Sync-Ope-proto-rescue:POT-Sync-Ope-proto -> Sync-Ope-proto-rescue:POT-Sync-Ope-proto-Sync-Ope-proto-rescue
- U1: symbol Sync-Ope-proto-rescue:AD8072-Sync-Ope-proto -> Sync-Ope-proto-rescue:AD8072-Sync-Ope-proto-Sync-Ope-proto-rescue
- U2: symbol Sync-Ope-proto-rescue:LM1881-Sync-Ope-proto -> Sync-Ope-proto-rescue:LM1881-Sync-Ope-proto-Sync-Ope-proto-rescue
- U5: symbol Sync-Ope-proto-rescue:LT1251-Sync-Ope-proto -> Sync-Ope-proto-rescue:LT1251-Sync-Ope-proto-Sync-Ope-proto-rescue
Changed lines of the file:
@@
 $EndDescr
 $Comp
-L Sync-Ope-proto-rescue:AD8072-Sync-Ope-proto U1
+L Sync-Ope-proto-rescue:AD8072-Sync-Ope-proto-Sync-Ope-proto-rescue U1
 U 1 1 5DB6BAB3
 P 2750 1575
@@
 $EndComp
 $Comp
-L Sync-Ope-proto-rescue:AD8072-Sync-Ope-proto U1
+L Sync-Ope-proto-rescue:AD8072-Sync-Ope-proto-Sync-Ope-proto-rescue U1
 U 2 1 5DB6BB03
 P 3025 2725
@@
 $EndComp
 $Comp
-L Sync-Ope-proto-rescue:GND-Sync-Ope-proto #PWR04
+L Sync-Ope-proto-rescue:GND-Sync-Ope-proto-Sync-Ope-proto-rescue #PWR04
 U 1 1 5DB6BD48
 P 1400 1925
@@
 $EndComp
 $Comp
-L Sync-Ope-proto-rescue:R-Sync-Ope-proto R4
+L Sync-Ope-proto-rescue:R-Sync-Ope-proto-Sync-Ope-proto-rescue R4
 U 1 1 5DB6BE2D
 P 2300 1675
@@
 $EndComp
 $Comp
-L Sync-Ope-proto-rescue:R-Sync-Ope-proto R6
+L Sync-Ope-proto-rescue:R-Sync-Ope-proto-Sync-Ope-proto-rescue R6
 U 1 1 5DB6BE5E
 P 2575 2825
@@
 $EndComp
 $Comp
-L Sync-Ope-proto-rescue:+5V-Sync-Ope-proto #PWR010
+L Sync-Ope-proto-rescue:+5V-Sync-Ope-proto-Sync-Ope-proto-rescue #PWR010
 U 1 1 5DB6BEB9
 P 2650 1200
@@
 	2650 1200 2650 1275
 $Comp
-L Sync-Ope-proto-rescue:+5V-Sync-Ope-proto #PWR014
+L Sync-Ope-proto-rescue:+5V-Sync-Ope-proto-Sync-Ope-proto-rescue #PWR014
 U 1 1 5DB6BEEB
 P 2925 2350
@@
 	2425 3100 2425 2825
 $Comp
-L Sync-Ope-proto-rescue:-5V-Sync-Ope-proto #PWR9
+L Sync-Ope-proto-rescue:-5V-Sync-Ope-proto-Sync-Ope-proto-rescue #PWR9
 U 1 1 5DB6C058
 P 2425 2000
@@
 	2425 1875 2425 2000
 $Comp
-L Sync-Ope-proto-rescue:-5V-Sync-Ope-proto #PWR12
+L Sync-Ope-proto-rescue:-5V-Sync-Ope-proto-Sync-Ope-proto-rescue #PWR12
 U 1 1 5DB6C0D6
 P 2725 3200
@@
 	2725 3025 2725 3200
 $Comp
-L Sync-Ope-proto-rescue:GND-Sync-Ope-proto #PWR016
+L Sync-Ope-proto-rescue:GND-Sync-Ope-proto-Sync-Ope-proto-rescue #PWR016
 U 1 1 5DB6C59E
 P 3975 2925
@@
 $EndComp
 $Comp
-L Sync-Ope-proto-rescue:R-Sync-Ope-proto R8
+L Sync-Ope-proto-rescue:R-Sync-Ope-proto-Sync-Ope-proto-rescue R8
 U 1 1 5DB6C5C2
 P 3725 2725
@@
 VIDEO_TO_SYNC
 $Comp
-L Sync-Ope-proto-rescue:LM1881-Sync-Ope-proto U2
+L Sync-Ope-proto-rescue:LM1881-Sync-Ope-proto-Sync-Ope-proto-rescue U2
 U 1 1 5DB6CFDE
 P 3350 4675
@@
 $EndComp
 $Comp
-L Sync-Ope-proto-rescue:C-Sync-Ope-proto C3
+L Sync-Ope-proto-rescue:C-Sync-Ope-proto-Sync-Ope-proto-rescue C3
 U 1 1 5DB6D144
 P 2325 4375
@@
 NoConn ~ 4000 4375
 $Comp
-L Sync-Ope-proto-rescue:+5V-Sync-Ope-proto #PWR018
+L Sync-Ope-proto-rescue:+5V-Sync-Ope-proto-Sync-Ope-proto-rescue #PWR018
 U 1 1 5DB6D3A9
 P 4125 3800
@@
 	4125 3800 4125 4275
 $Comp
-L Sync-Ope-proto-rescue:GND-Sync-Ope-proto #PWR011
+L Sync-Ope-proto-rescue:GND-Sync-Ope-proto-Sync-Ope-proto-rescue #PWR011
 U 1 1 5DB6D40B
 P 2700 5150
@@
 $EndComp
 $Comp
-L Sync-Ope-proto-rescue:R-Sync-Ope-proto R9
+L Sync-Ope-proto-rescue:R-Sync-Ope-proto-Sync-Ope-proto-rescue R9
 U 1 1 5DB6D49F
 P 4350 4475
@@
 $EndComp
 $Comp
-L Sync-Ope-proto-rescue:C-Sync-Ope-proto C4
+L Sync-Ope-proto-rescue:C-Sync-Ope-proto-Sync-Ope-proto-rescue C4
 U 1 1 5DB6D4EA
 P 4350 4300
@@
 	4200 4475 4200 4300
 $Comp
-L Sync-Ope-proto-rescue:GND-Sync-Ope-proto #PWR020
+L Sync-Ope-proto-rescue:GND-Sync-Ope-proto-Sync-Ope-proto-rescue #PWR020
 U 1 1 5DB6D6AF
 P 4650 4825
@@
 	4000 4700 4925 4700
 $Comp
-L Sync-Ope-proto-rescue:LT1251-Sync-Ope-proto U5
+L Sync-Ope-proto-rescue:LT1251-Sync-Ope-proto-Sync-Ope-proto-rescue U5
 U 1 1 5DB717D4
 P 8375 2525
@@
 $EndComp
 $Comp
-L Sync-Ope-proto-rescue:GND-Sync-Ope-proto #PWR024
+L Sync-Ope-proto-rescue:GND-Sync-Ope-proto-Sync-Ope-proto-rescue #PWR024
 U 1 1 5DB71BE2
 P 7075 2600
@@
 $EndComp
 $Comp
-L Sync-Ope-proto-rescue:R-Sync-Ope-proto R13
+L Sync-Ope-proto-rescue:R-Sync-Ope-proto-Sync-Ope-proto-rescue R13
 U 1 1 5DB71E30
 P 7575 1400
@@
 	9325 1825 8875 1825
 $Comp
-L Sync-Ope-proto-rescue:R-Sync-Ope-proto R15
+L Sync-Ope-proto-rescue:R-Sync-Ope-proto-Sync-Ope-proto-rescue R15
 U 1 1 5DB72713
 P 7725 1925
@@
 $EndComp
 $Comp
-L Sync-Ope-proto-rescue:R-Sync-Ope-proto R17
+L Sync-Ope-proto-rescue:R-Sync-Ope-proto-Sync-Ope-proto-rescue R17
 U 1 1 5DB72840
 P 9175 1925
@@
 NoConn ~ 8875 2125
 $Comp
-L Sync-Ope-proto-rescue:GND-Sync-Ope-proto #PWR033
+L Sync-Ope-proto-rescue:GND-Sync-Ope-proto-Sync-Ope-proto-rescue #PWR033
 U 1 1 5DB72D25
 P 9525 2625
@@
 NoConn ~ 7875 2325
 $Comp
-L Sync-Ope-proto-rescue:-5V-Sync-Ope-proto #PWR26
+L Sync-Ope-proto-rescue:-5V-Sync-Ope-proto-Sync-Ope-proto-rescue #PWR26
 U 1 1 5DB72F1F
 P 7875 2750
@@
 $EndComp
 $Comp
-L Sync-Ope-proto-rescue:+5V-Sync-Ope-proto #PWR034
+L Sync-Ope-proto-rescue:+5V-Sync-Ope-proto-Sync-Ope-proto-rescue #PWR034
 U 1 1 5DB73053
 P 9850 1775
@@
 $EndComp
 $Comp
-L Sync-Ope-proto-rescue:R-Sync-Ope-proto R18
+L Sync-Ope-proto-rescue:R-Sync-Ope-proto-Sync-Ope-proto-rescue R18
 U 1 1 5DB7312B
 P 9325 2125
@@
 $EndComp
 $Comp
-L Sync-Ope-proto-rescue:R-Sync-Ope-proto R19
+L Sync-Ope-proto-rescue:R-Sync-Ope-proto-Sync-Ope-proto-rescue R19
 U 1 1 5DB73D34
 P 9675 2025
@@
 	7450 1925 7575 1925
 $Comp
-L Sync-Ope-proto-rescue:GND-Sync-Ope-proto #PWR035
+L Sync-Ope-proto-rescue:GND-Sync-Ope-proto-Sync-Ope-proto-rescue #PWR035
 U 1 1 5DB75A8A
 P 10600 2800
@@
 $EndComp
 $Comp
-L Sync-Ope-proto-rescue:R-Sync-Ope-proto R20
+L Sync-Ope-proto-rescue:R-Sync-Ope-proto-Sync-Ope-proto-rescue R20
 U 1 1 5DB75A90
 P 10250 2525
@@
 Power Supply
 $Comp
-L Sync-Ope-proto-rescue:PWR_FLAG-Sync-Ope-proto #FLG02
+L Sync-Ope-proto-rescue:PWR_FLAG-Sync-Ope-proto-Sync-Ope-proto-rescue #FLG02
 U 1 1 5DB7A4FE
 P 4725 6000
@@
 $EndComp
 $Comp
-L Sync-Ope-proto-rescue:PWR_FLAG-Sync-Ope-proto #FLG03
+L Sync-Ope-proto-rescue:PWR_FLAG-Sync-Ope-proto-Sync-Ope-proto-rescue #FLG03
 U 1 1 5DB7A70A
 P 4400 6200
@@
 $EndComp
 $Comp
-L Sync-Ope-proto-rescue:PWR_FLAG-Sync-Ope-proto #FLG01
+L Sync-Ope-proto-rescue:PWR_FLAG-Sync-Ope-proto-Sync-Ope-proto-rescue #FLG01
 U 1 1 5DB7A8B8
 P 4725 5800
@@
 $EndComp
 $Comp
-L Sync-Ope-proto-rescue:POT-Sync-Ope-proto RV1
+L Sync-Ope-proto-rescue:POT-Sync-Ope-proto-Sync-Ope-proto-rescue RV1
 U 1 1 5DB76F3B
 P 6725 2025
@@
 $EndComp
 $Comp
-L Sync-Ope-proto-rescue:R-Sync-Ope-proto R12
+L Sync-Ope-proto-rescue:R-Sync-Ope-proto-Sync-Ope-proto-rescue R12
 U 1 1 5DB7F722
 P 7375 1825
@@
 	6725 2175 6725 2225
 $Comp
-L Sync-Ope-proto-rescue:R-Sync-Ope-proto R11
+L Sync-Ope-proto-rescue:R-Sync-Ope-proto-Sync-Ope-proto-rescue R11
 U 1 1 5DB80EB4
 P 7275 2025
@@
 	1550 1475 1650 1475
 $Comp
-L Sync-Ope-proto-rescue:R-Sync-Ope-proto R1
+L Sync-Ope-proto-rescue:R-Sync-Ope-proto-Sync-Ope-proto-rescue R1
 U 1 1 5DB6BD67
 P 1650 1625
@@
 	7425 2025 7875 2025
 $Comp
-L Sync-Ope-proto-rescue:C-Sync-Ope-proto C5
+L Sync-Ope-proto-rescue:C-Sync-Ope-proto-Sync-Ope-proto-rescue C5
 U 1 1 5DB9B36B
 P 9000 2225
@@
 	9000 2025 9100 2025
 $Comp
-L Sync-Ope-proto-rescue:GND-Sync-Ope-proto #PWR032
+L Sync-Ope-proto-rescue:GND-Sync-Ope-proto-Sync-Ope-proto-rescue #PWR032
 U 1 1 5DBAB6B3
 P 9000 2625
@@
 Signal Blanking
 $Comp
-L Sync-Ope-proto-rescue:+5V-Sync-Ope-proto #PWR030
+L Sync-Ope-proto-rescue:+5V-Sync-Ope-proto-Sync-Ope-proto-rescue #PWR030
 U 1 1 5DCF1AA3
 P 8700 3950
@@
 $EndComp
 $Comp
-L Sync-Ope-proto-rescue:-5V-Sync-Ope-proto #PWR31
+L Sync-Ope-proto-rescue:-5V-Sync-Ope-proto-Sync-Ope-proto-rescue #PWR31
 U 1 1 5DD5D6B4
 P 8800 6075
@@
 	7075 1825 7075 2225
 $Comp
-L Sync-Ope-proto-rescue:GND-Sync-Ope-proto #PWR029
+L Sync-Ope-proto-rescue:GND-Sync-Ope-proto-Sync-Ope-proto-rescue #PWR029
 U 1 1 5DCF6ECA
 P 8300 5900
@@
 $EndComp
 $Comp
-L Sync-Ope-proto-rescue:+5V-Sync-Ope-proto #PWR025
+L Sync-Ope-proto-rescue:+5V-Sync-Ope-proto-Sync-Ope-proto-rescue #PWR025
 U 1 1 5DE95345
 P 7675 4625
@@
 $EndComp
 $Comp
-L Sync-Ope-proto-rescue:+5V-Sync-Ope-proto #PWR027
+L Sync-Ope-proto-rescue:+5V-Sync-Ope-proto-Sync-Ope-proto-rescue #PWR027
 U 1 1 5DE47489
 P 8100 3550
@@
 	2550 5075 2700 5075
 $Comp
-L Sync-Ope-proto-rescue:R-Sync-Ope-proto R5
+L Sync-Ope-proto-rescue:R-Sync-Ope-proto-Sync-Ope-proto-rescue R5
 U 1 1 5E0F4BED
 P 2550 4925
@@
 	5325 6500 5325 6750
 $Comp
-L Sync-Ope-proto-rescue:Conn_Rca-Sync-Ope-proto J1
+L Sync-Ope-proto-rescue:Conn_Rca-Sync-Ope-proto-Sync-Ope-proto-rescue J1
 U 1 1 5E12D073
 P 1400 1475
@@
 $EndComp
 $Comp
-L Sync-Ope-proto-rescue:Conn_Rca-Sync-Ope-proto J6
+L Sync-Ope-proto-rescue:Conn_Rca-Sync-Ope-proto-Sync-Ope-proto-rescue J6
 U 1 1 5E165212
 P 10600 2525

Commit message: update circuit design to 0.2
Parts:
- added J10, J9: rca, lib_fp:RCJ-024, symbol Connector:Conn_Coaxial
- C1, C2, C3, C4, C5, C6, C7, C8, C9: footprint Capacitor_THT:C_Axial_L3.8mm_D2.6mm_P7.50mm_Horizontal -> Capacitor_THT:C_Disc_D4.3mm_W1.9mm_P5.00mm
- C10, C11, C12, C13: footprint Capacitor_THT:CP_Radial_D5.0mm_P2.50mm -> Capacitor_THT:CP_Radial_D7.5mm_P2.50mm
- D2, D3: value D -> 1n4148
- D4, D5: footprint Diode_THT:D_DO-35_SOD27_P7.62mm_Horizontal -> Diode_THT:D_DO-35_SOD27_P10.16mm_Horizontal
- J1: value VIDEO_INPUT -> rca; footprint project_parts:RCJ-024 -> lib_fp:RCJ-024; symbol Sync-Ope-proto-rescue:Conn_Rca-Sync-Ope-proto-Sync-Ope-proto-rescue -> Connector:Conn_Coaxial
- J3: value VIDEO_SEND -> mono_jack
- J4: value VIDEO_RETURN -> mono_jack
- J5: value CV_IN -> mono_jack
- J6: value VIDEO_OUTPUT -> rca; footprint project_parts:RCJ-024 -> lib_fp:RCJ-024; symbol Sync-Ope-proto-rescue:Conn_Rca-Sync-Ope-proto-Sync-Ope-proto-rescue -> Connector:Conn_Coaxial
- J7: symbol Connector:Barrel_Jack -> Connector:Barrel_Jack_Switch
- R1, R10, R11, R12, R13, R14, R15, R16, R17, R18, R19, R2, R20, R3, R4, R5, R6, R7, R8, R9: footprint Resistor_THT:R_Axial_DIN0204_L3.6mm_D1.6mm_P5.08mm_Horizontal -> Resistor_THT:R_Axial_DIN0204_L3.6mm_D1.6mm_P7.62mm_Horizontal
- U1, U2: footprint Package_DIP:DIP-8_W7.62mm -> Package_DIP:DIP-8_W7.62mm_LongPads
- U3, U4: footprint Package_TO_SOT_THT:TO-220-3_Horizontal_TabUp -> Package_TO_SOT_THT:TO-220-3_Vertical
- U5: footprint Package_DIP:DIP-14_W7.62mm_Socket -> Package_DIP:DIP-14_W7.62mm_Socket_LongPads
- U6: footprint Package_DIP:DIP-16_W7.62mm_Socket -> Package_DIP:DIP-16_W7.62mm_LongPads
Connections:
- wire segments 214 -> 216
- no-connect marks 12 -> 13

Commit message: latest revision
Parts:
- C12, C13: value 200u -> 220u
Changed lines of the file:
@@
 Wire Wire Line
 	2175 1475 2450 1475
-Text GLabel 1775 2275 3    60   Input ~ 0
+Text GLabel 1775 2275 0    60   Input ~ 0
 VIDEO_TO_SYNC
 Wire Wire Line
@@
 P 4175 5900
 F 0 "C12" H 4263 5946 50  0000 L CNN
-F 1 "200u" H 4263 5855 50  0000 L CNN
+F 1 "220u" H 4263 5855 50  0000 L CNN
 F 2 "Capacitor_THT:CP_Radial_D7.5mm_P2.50mm" H 4175 5900 50  0001 C CNN
 F 3 "~" H 4175 5900 50  0001 C CNN
@@
 P 4175 6100
 F 0 "C13" H 4263 6146 50  0000 L CNN
-F 1 "200u" H 4263 6055 50  0000 L CNN
+F 1 "220u" H 4263 6055 50  0000 L CNN
 F 2 "Capacitor_THT:CP_Radial_D7.5mm_P2.50mm" H 4175 6100 50  0001 C CNN
 F 3 "~" H 4175 6100 50  0001 C CNN

Commit message: Add files via upload
Parts:
- removed C1: 100n, Capacitor_THT:C_Disc_D4.3mm_W1.9mm_P5.00mm, symbol Device:C
- added C14: 1nF, symbol Sync-Ope-proto-rescue:C-Device
- added CD4069: delay clamping signal, symbol Sync-Ope-proto-rescue:CD4069
- added R21: 3.3K, symbol Sync-Ope-proto-rescue:R-Device
- C10, C11: symbol Device:CP -> Sync-Ope-proto-rescue:CP-Device
- C12, C13: symbol Device:CP_Small -> Sync-Ope-proto-rescue:CP_Small-Device
- C2, C6, C7, C8, C9: symbol Device:C -> Sync-Ope-proto-rescue:C-Device
- D1: symbol Device:LED -> Sync-Ope-proto-rescue:LED-Device
- D2, D3, D4, D5: symbol Device:D -> Sync-Ope-proto-rescue:D-Device
- D6: symbol Device:D_Zener -> Sync-Ope-proto-rescue:D_Zener-Device
- D7: symbol Device:D_Schottky -> Sync-Ope-proto-rescue:D_Schottky-Device
- J1, J10, J6, J9: symbol Connector:Conn_Coaxial -> Sync-Ope-proto-rescue:Conn_Coaxial-Connector
- J2: symbol Connector_Generic:Conn_02x08_Odd_Even -> Sync-Ope-proto-rescue:Conn_02x08_Odd_Even-Connector_Generic
- J3, J4, J5: symbol Connector:AudioJack2_SwitchT -> Sync-Ope-proto-rescue:AudioJack2_SwitchT-Connector
- J7: symbol Connector:Barrel_Jack_Switch -> Sync-Ope-proto-rescue:Barrel_Jack_Switch-Connector
- J8: symbol Connector:Conn_01x03_Female -> Sync-Ope-proto-rescue:Conn_01x03_Female-Connector
- R10, R14, R16, R2, R3, R7: symbol Device:R -> Sync-Ope-proto-rescue:R-Device
- U3: symbol Regulator_Linear:L7805 -> Sync-Ope-proto-rescue:L7805-Regulator_Linear
- U4: symbol Regulator_Linear:L7905 -> Sync-Ope-proto-rescue:L7905-Regulator_Linear
- U6: symbol 4xxx:4053 -> Sync-Ope-proto-rescue:4053-4xxx
Connections:
- wire segments 216 -> 240
- no-connect marks 13 -> 14
Other:
- note added: "CV IN (0_1V)"
- note added: "VIDEO IN"
- note added: "VIDEO OUT"
- note added: "VIDEO RETURN"
- note added: "VIDEO SEND"
- moved on the sheet: R14, R16, R2, R3, R4

Commit message: circuit revision 0.3
Parts:
- removed C14: 1nF, symbol Sync-Ope-proto-rescue:C-Device
- removed C3, C4: 100n, Capacitor_THT:C_Disc_D4.3mm_W1.9mm_P5.00mm, symbol Sync-Ope-proto-rescue:C-Sync-Ope-proto-Sync-Ope-proto-rescue
- removed CD4069: delay clamping signal, symbol Sync-Ope-proto-rescue:CD4069
- removed D1: video signal indicator LED, LED_THT:LED_D3.0mm, symbol Sync-Ope-proto-rescue:LED-Device
- removed D2, D3: 1n4148, Diode_THT:D_DO-35_SOD27_P7.62mm_Horizontal, symbol Sync-Ope-proto-rescue:D-Device
- removed R10: 100k, Resistor_THT:R_Axial_DIN0204_L3.6mm_D1.6mm_P7.62mm_Horizontal, symbol Sync-Ope-proto-rescue:R-Device
- removed R14: 10k, Resistor_THT:R_Axial_DIN0204_L3.6mm_D1.6mm_P7.62mm_Horizontal, symbol Sync-Ope-proto-rescue:R-Device
- removed R16: 39k, Resistor_THT:R_Axial_DIN0204_L3.6mm_D1.6mm_P7.62mm_Horizontal, symbol Sync-Ope-proto-rescue:R-Device
- removed R21: 3.3K, symbol Sync-Ope-proto-rescue:R-Device
- removed R3: 220, Resistor_THT:R_Axial_DIN0204_L3.6mm_D1.6mm_P7.62mm_Horizontal, symbol Sync-Ope-proto-rescue:R-Device
- removed R5: 1k, Resistor_THT:R_Axial_DIN0204_L3.6mm_D1.6mm_P7.62mm_Horizontal, symbol Sync-Ope-proto-rescue:R-Sync-Ope-proto-Sync-Ope-proto-rescue
- removed R9: 680k, Resistor_THT:R_Axial_DIN0204_L3.6mm_D1.6mm_P7.62mm_Horizontal, symbol Sync-Ope-proto-rescue:R-Sync-Ope-proto-Sync-Ope-proto-rescue
- removed U2: LM1881, Package_DIP:DIP-8_W7.62mm_LongPads, symbol Sync-Ope-proto-rescue:LM1881-Sync-Ope-proto-Sync-Ope-proto-rescue
- removed U6: CD4053BE, Package_DIP:DIP-16_W7.62mm_LongPads, symbol Sync-Ope-proto-rescue:4053-4xxx
- added C14, C15, C16, C17, C18, C19: 0.1u, Capacitor_THT:C_Disc_D4.3mm_W1.9mm_P5.00mm, symbol Device:C_Small
- added R3: 510, Resistor_THT:R_Axial_DIN0204_L3.6mm_D1.6mm_P7.62mm_Horizontal, symbol Sync-Ope-proto-rescue:R-Sync-Ope-proto-Sync-Ope-proto-rescue
- added R5: 39k, Resistor_THT:R_Axial_DIN0204_L3.6mm_D1.6mm_P7.62mm_Horizontal, symbol Sync-Ope-proto-rescue:R-Device
- C2, C5, C7, C9: value 100n -> 0.1u
- C6, C8: value 330n -> 0.33u
- D7: value schottky -> bat46
- J1, J10, J6, J9: footprint lib_fp:RCJ-024 -> lib_fp:tht_vertical_rca
- J2: value euro_power -> europower
- J3, J4, J5: value mono_jack -> mono_jack_3.5mm
- J7: value AC_POWER -> barrel_jack
- R18: symbol Sync-Ope-proto-rescue:R-Sync-Ope-proto-Sync-Ope-proto-rescue -> Device:R
- RV1: value 10k -> 10k_pot
- U1: footprint Package_DIP:DIP-8_W7.62mm_LongPads -> lib_fp:DIP-SOIC-8
Connections:
- net +5V: now also C14.1, C15.1, C16.1, C17.1, R5.1
- net -5V: now also C18.2, C19.2
- net GND: now also R12.1, C14.2, C15.2, C16.2, C17.2, C18.1, C19.1; no longer J4.TN, R12.2
- net at D6.1 (K), D7.1 (K), U5.1 (IN_1): now also R12.2, R13.1; no longer R12.1, R13.2
- net blanking/return_blank: now reaches J4.T, J9.1 (In)
- net blanking/return_blank: now also R13.2; no longer R13.1
- net at J5.TN: now also R5.2
- net blanking/control_blank: now reaches J5.T
- net ADDED_SYNC renamed blanking/control_pulse
- net DRY_BLANKED_SIGNAL renamed blanking/input_blank
- net VIDEO_TO_SYNC renamed blanking/video_in
- net blanking/video_in: now also R3.2; no longer U1.3 (+)
- new net: R3.1, U1.3 (+)
- no-connect marks 14 -> 12
Other:
- note added: "DRY/WET"
- note removed: "Signal Blanking"
- note removed: "Video Sync Seperator"
- moved on the sheet: C10, C11, C12, C13, C2, C5, C6, C7, C8, C9, D4, D5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

Commit message: working on v0.4.0
Parts:
- added C23: 0.1u, Capacitor_THT:C_Disc_D4.3mm_W1.9mm_P5.00mm, symbol Device:C_Small
- RV1: footprint Potentiometer_THT:Potentiometer_Alps_RK09K_Single_Vertical -> lib_fp:Potentiometer_Vertical_Large
- U4: renamed from U5; footprint Package_DIP:DIP-14_W7.62mm_Socket_LongPads -> lib_fp:DIP+SOIC_14
- renumbered C12 to C1, C14 to C10, C18 to C11, C15 to C12, C19 to C13, C16 to C14, C17 to C15, C5 to C16, C13 to C2, C6 to C3, C2 to C4, C10 to C5, C7 to C6, C8 to C7, C11 to C8, D4 to D1, D5 to D2, D6 to D3, D7 to D4, J6 to J10, J7 to J2, J2 to J3, J5 to J4, J3 to J5, J10 to J6, J8 to J7, J4 to J8, R12 to R10, R15 to R12, R17 to R13, R18 to R14, R19 to R15, R20 to R16, R6 to R4, R4 to R5, R7 to R6, R8 to R7, R5 to R8, R13 to R9, U3 to U2, U4 to U3
Connections:
- net +5V: now also C23.1
- net GND: now also C23.2
