File: kicad-files/blanking.sch (KiCad schematic (older format))
At the start: 11 parts, among them U2 74HC4538, U6 LM1881, U7 CD4053B

Commit message: working on v0.4.0
Parts:
- added C19, C21: 1nf, Capacitor_THT:C_Disc_D4.7mm_W2.5mm_P5.00mm, symbol Device:C_Small
- added C22: 1uf, Capacitor_THT:C_Disc_D4.7mm_W2.5mm_P5.00mm, symbol Device:C_Small
- added R19: 10k, Resistor_THT:R_Axial_DIN0204_L3.6mm_D1.6mm_P7.62mm_Horizontal, symbol Device:R
- added R21: 75k, Resistor_THT:R_Axial_DIN0204_L3.6mm_D1.6mm_P7.62mm_Horizontal, symbol Device:R
- added R22: 22k, Resistor_THT:R_Axial_DIN0204_L3.6mm_D1.6mm_P7.62mm_Horizontal, symbol Device:R
- added RV2, RV4: 5k_trim, lib_fp:tht_vertical_trim_3362, symbol Device:R_POT
- added RV5: 10k_trim, lib_fp:tht_vertical_trim_3362, symbol Device:R_POT
- added unit 1 of U5
- added unit 2 of U5
- added unit 3 of U6
- added unit 2 of U6
- C20: renamed from C1; value 0.001u -> 0.1u
- R20: renamed from R9; value 10k -> 12k
- RV3: renamed from RV2; value 5k_trim -> 10k_trim
- U8: renamed from U7; symbol Analog_Switch:CD4053B -> Sync-Ope-proto-rescue:CD4053B-Analog_Switch
- renumbered C3 to C17, C4 to C18, D1 to D5, R14 to R17, R16 to R18, U2 to U5, U2 to U6, U6 to U7
Connections:
- net +5V: now also RV2.1, RV4.1, RV5.1, U5.13 (~CD), U6.13 (~CD), U6.16 (VDD)
- net GND: now also U5.12 (B), U5.4 (B), U6.12 (B), U6.8 (VSS)
- net c_blanking: now reaches U8.10 (B), U8.11 (A), U8.9 (C)
- net c_blanking: now also U5.10 (Q); no longer U6.6 (Q)
- net at U6.5 (~A): now also D5.2 (A), U7.3 (FRAME); no longer U7.1 (CSYNC)
- new net: U6.11 (~A), U6.6 (Q)
- new net: U5.5 (~A), U7.1 (CSYNC)
- new net: C22.2, R22.1, U6.14 (RxCx)
- new net: C22.1, U6.15 (Cx)
- new net: R22.2, RV5.2
- new net: C19.1, U5.1 (Cx)
- new net: C19.2, R19.1, U5.2 (RxCx)
- new net: U5.11 (~A), U5.6 (Q)
- new net: R19.2, RV2.2
- new net: C21.2, R21.1, U5.14 (RxCx)
- new net: C21.1, U5.15 (Cx)
- new net: R21.2, RV4.2
- new net v_blanking: U5.3 (~CD), U6.10 (Q)
- no-connect marks 6 -> 12
Other:
- moved on the sheet: C17, C18, C20, D5, R17, R18, R20, RV3, U5C, U6A, U7, U8
