File: hardware/Sync-Ope-proto.kicad_pcb (KiCad board)
At the start: 2 copper layers, 100 x 100 mm, 77 parts, among them J1 rca, J10 rca, J2 barrel_jack, J3 europower, J4 mono_jack_3.5mm, J5 mono_jack_3.5mm, J6 rca, J7 diy_power_header, J8 mono_jack_3.5mm, J9 rca, U1 AD8072, U2 L7805, U3 L7905, U4 LT1251, U5 74HC4538, U6 74HC4538, U7 LM1881, U8 CD4053B

Commit message: update circuit
Parts:
- J2: footprint Connector_BarrelJack:BarrelJack_Horizontal -> lib_fp:BarrelJack_Horizontal
- J4, J5, J8: footprint Connector_Audio:Jack_3.5mm_QingPu_WQP-PJ398SM_Vertical_CircularHoles -> lib_fp:Jack_3.5mm_QingPu_WQP-PJ398SM_Vertical_CircularHoles
