File: panel/default_panel/default_panel.kicad_pcb (KiCad board)
At the start: 2 copper layers, 100 x 100 mm, 4 parts

Commit message: add panel stuff
Parts:
- removed REF** (x4): MountingHole_3.2mm_M3, MountingHole:MountingHole_3.2mm_M3
Other:
- outline, holes or cut-outs redrawn
- board text added: "sync_ope default panel - mk_i for v1_0_1 based on Gael Jaton design updated by cyberboy666"
- board text removed: "sync_ope panel for v1_0_1 - mk_i based on Gael Jaton design updated by cyberboy666"
Changed lines of the file:
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@@
       (drillshape 0)
       (scaleselection 1)
-      (outputdirectory "./default_panel_for_v1_0_1_mk_i")
+      (outputdirectory "./sync_ope_default_panel_for_v1_0_1_mk_ii")
     )
   )
   (net 0 "")
-  (footprint "MountingHole:MountingHole_3.2mm_M3" (layer "F.Cu")
-    (at 196.6 146.5)
-    (descr "Mounting Hole 3.2mm, no annular, M3")
-    (tags "mounting hole 3.2mm no annular m3")
-    (attr exclude_from_pos_files exclude_from_bom)
-    (fp_text reference "REF**" (at 0 -4.2) (layer "F.SilkS") hide
-      (effects (font (size 1 1) (thickness 0.15)))
-    )
-    (fp_text value "MountingHole_3.2mm_M3" (at 0 4.2) (layer "F.Fab") hide
-      (effects (font (size 1 1) (thickness 0.15)))
-    )
-    (fp_text user "${REFERENCE}" (at 0 0) (layer "F.Fab")
-      (effects (font (size 1 1) (thickness 0.15)))
-    )
-    (fp_circle (center 0 0) (end 3.2 0) (layer "Cmts.User") (width 0.15) (fill none))
-    (fp_circle (center 0 0) (end 3.45 0) (layer "F.CrtYd") (width 0.05) (fill none))
-    (pad "" np_thru_hole circle (at 0 0) (size 3.2 3.2) (drill 3.2) (layers *.Cu *.Mask))
-  )
-  (footprint "MountingHole:MountingHole_3.2mm_M3" (layer "F.Cu")
-    (at 196.5 53.5)
-    (descr "Mounting Hole 3.2mm, no annular, M3")
-    (tags "mounting hole 3.2mm no annular m3")
-    (attr exclude_from_pos_files exclude_from_bom)
-    (fp_text reference "REF**" (at 0 -4.2) (layer "F.SilkS") hide
-      (effects (font (size 1 1) (thickness 0.15)))
-    )
-    (fp_text value "MountingHole_3.2mm_M3" (at 0 4.2) (layer "F.Fab") hide
-      (effects (font (size 1 1) (thickness 0.15)))
-    )
-    (fp_text user "${REFERENCE}" (at 0 0) (layer "F.Fab")
-      (effects (font (size 1 1) (thickness 0.15)))
-    )
-    (fp_circle (center 0 0) (end 3.2 0) (layer "Cmts.User") (width 0.15) (fill none))
-    (fp_circle (center 0 0) (end 3.45 0) (layer "F.CrtYd") (width 0.05) (fill none))
-    (pad "" np_thru_hole circle (at 0 0) (size 3.2 3.2) (drill 3.2) (layers *.Cu *.Mask))
-  )
-  (footprint "MountingHole:MountingHole_3.2mm_M3" (layer "F.Cu")
-    (at 103.5 146.5)
-    (descr "Mounting Hole 3.2mm, no annular, M3")
-    (tags "mounting hole 3.2mm no annular m3")
-    (attr exclude_from_pos_files exclude_from_bom)
-    (fp_text reference "REF**" (at 0 -4.2) (layer "F.SilkS") hide
-      (effects (font (size 1 1) (thickness 0.15)))
-    )
-    (fp_text value "MountingHole_3.2mm_M3" (at 0 4.2) (layer "F.Fab") hide
-      (effects (font (size 1 1) (thickness 0.15)))
-    )
-    (fp_text user "${REFERENCE}" (at 0 0) (layer "F.Fab")
-      (effects (font (size 1 1) (thickness 0.15)))
-    )
-    (fp_circle (center 0 0) (end 3.2 0) (layer "Cmts.User") (width 0.15) (fill none))
-    (fp_circle (center 0 0) (end 3.45 0) (layer "F.CrtYd") (width 0.05) (fill none))
-    (pad "" np_thru_hole circle (at 0 0) (size 3.2 3.2) (drill 3.2) (layers *.Cu *.Mask))
-  )
-  (footprint "MountingHole:MountingHole_3.2mm_M3" (layer "F.Cu")
-    (at 103.4 53.5)
-    (descr "Mounting Hole 3.2mm, no annular, M3")
-    (tags "mounting hole 3.2mm no annular m3")
-    (attr exclude_from_pos_files exclude_from_bom)
-    (fp_text reference "REF**" (at 0 -4.2) (layer "F.SilkS") hide
-      (effects (font (size 1 1) (thickness 0.15)))
-    )
-    (fp_text value "MountingHole_3.2mm_M3" (at 0 4.2) (layer "F.Fab") hide
-      (effects (font (size 1 1) (thickness 0.15)))
-    )
-    (fp_text user "${REFERENCE}" (at 0 0) (layer "F.Fab")
-      (effects (font (size 1 1) (thickness 0.15)))
-    )
-    (fp_circle (center 0 0) (end 3.2 0) (layer "Cmts.User") (width 0.15) (fill none))
-    (fp_circle (center 0 0) (end 3.45 0) (layer "F.CrtYd") (width 0.05) (fill none))
-    (pad "" np_thru_hole circle (at 0 0) (size 3.2 3.2) (drill 3.2) (layers *.Cu *.Mask))
-  )
-  (gr_line (start 111.15 134.65) (end 110.1 128.4) (layer "F.SilkS") (width 0.5))
+  (gr_line (start 110.96 133.6) (end 110.1 128.4) (layer "F.SilkS") (width 0.5))
   (gr_line (start 149.8 108.4) (end 149.8 104.55) (layer "F.SilkS") (width 0.5))
-  (gr_line (start 189.975 128.325) (end 188.925 134.575) (layer "F.SilkS") (width 0.5))
+  (gr_line (start 189.975 128.325) (end 189.23 133) (layer "F.SilkS") (width 0.5))
   (gr_line (start 100 150) (end 100 50) (layer "Edge.Cuts") (width 0.05))
   (gr_circle (center 135.7 145.65) (end 137.7 145.65) (layer "Edge.Cuts") (width 0.05) (fill none))
@@
   (gr_circle (center 158.2 145.6) (end 160.2 145.6) (layer "Edge.Cuts") (width 0.05) (fill none))
   (gr_circle (center 135.7 131.65) (end 137.7 131.65) (layer "Edge.Cuts") (width 0.05) (fill none))
-  (gr_circle (center 113.15 60.05) (end 118.15 60.05) (layer "Edge.Cuts") (width 0.05) (fill none))
-  (gr_line (start 168.25 50) (end 200 50) (layer "Edge.Cuts") (width 0.05))
-  (gr_line (start 142.85 52.7) (end 142.85 50) (layer "Edge.Cuts") (width 0.05))
-  (gr_line (start 131.8 52.7) (end 142.85 52.7) (layer "Edge.Cuts") (width 0.05))
+  (gr_circle (center 103.5 53.5) (end 105.3 53.5) (layer "Edge.Cuts") (width 0.05) (fill none))
+  (gr_circle (center 113.15 60.05) (end 119.65 60.05) (layer "Edge.Cuts") (width 0.05) (fill none))
+  (gr_circle (center 196.5 146.5) (end 198.3 146.5) (layer "Edge.Cuts") (width 0.05) (fill none))
   (gr_circle (center 158.2 131.65) (end 160.2 131.65) (layer "Edge.Cuts") (width 0.05) (fill none))
-  (gr_line (start 157.2 52.7) (end 168.25 52.7) (layer "Edge.Cuts") (width 0.05))
-  (gr_circle (center 187.5 60.55) (end 192.5 60.55) (layer "Edge.Cuts") (width 0.05) (fill none))
-  (gr_line (start 100 50) (end 131.8 50) (layer "Edge.Cuts") (width 0.05))
-  (gr_line (start 131.8 50) (end 131.8 52.7) (layer "Edge.Cuts") (width 0.05))
-  (gr_line (start 157.2 50) (end 157.2 52.7) (layer "Edge.Cuts") (width 0.05))
-  (gr_line (start 157.2 50) (end 142.85 50) (layer "Edge.Cuts") (width 0.05))
+  (gr_circle (center 187.5 60.55) (end 194 60.55) (layer "Edge.Cuts") (width 0.05) (fill none))
+  (gr_circle (center 103.5 146.5) (end 105.3 146.5) (layer "Edge.Cuts") (width 0.05) (fill none))
+  (gr_line (start 100 50) (end 200 50) (layer "Edge.Cuts") (width 0.05))
   (gr_circle (center 150.25 89.5) (end 151.95 89.5) (layer "Edge.Cuts") (width 0.05) (fill none))
   (gr_circle (center 109.5 123.9) (end 113 123.9) (layer "Edge.Cuts") (width 0.05) (fill none))
-  (gr_circle (center 112.05 140.6) (end 117.05 140.6) (layer "Edge.Cuts") (width 0.05) (fill none))
+  (gr_circle (center 112.05 140.6) (end 118.55 140.6) (layer "Edge.Cuts") (width 0.05) (fill none))
   (gr_circle (center 190.5 124.4) (end 194 124.4) (layer "Edge.Cuts") (width 0.05) (fill none))
   (gr_circle (center 150 100.4) (end 153.5 100.4) (layer "Edge.Cuts") (width 0.05) (fill none))
   (gr_circle (center 150 113) (end 154 113) (layer "Edge.Cuts") (width 0.05) (fill none))
-  (gr_circle (center 188.55 140) (end 193.55 140) (layer "Edge.Cuts") (width 0.05) (fill none))
+  (gr_circle (center 188.55 140) (end 195.05 140) (layer "Edge.Cuts") (width 0.05) (fill none))
   (gr_circle (center 104.25 65.5) (end 104.25 65.5) (layer "Edge.Cuts") (width 0.05) (fill none))
-  (gr_line (start 168.25 52.7) (end 168.25 50) (layer "Edge.Cuts") (width 0.05))
+  (gr_circle (center 196.5 53.5) (end 198.3 53.5) (layer "Edge.Cuts") (width 0.05) (fill none))
   (gr_line (start 200 150) (end 100 150) (layer "Edge.Cuts") (width 0.05))
   (gr_text "underscores.shop" (at 150 86) (layer "B.SilkS")
     (effects (font (size 1.5 1.5) (thickness 0.3)) (justify mirror))
   )
-  (gr_text "sync_ope panel \nfor v1_0_1 - mk_i\nbased on Gael Jaton design\nupdated by cyberboy666" (at 198.35 74.1) (layer "B.SilkS")
+  (gr_text "sync_ope default panel - mk_i\nfor v1_0_1\nbased on Gael Jaton design\nupdated by cyberboy666" (at 198.35 74.1) (layer "B.SilkS")
     (effects (font (size 1.5 1.5) (thickness 0.3)) (justify left mirror))
   )
@@
     (effects (font (size 5 5) (thickness 0.5)) (justify mirror))
   )
-  (gr_text "VIDEO_IN" (at 112.5 52.35) (layer "F.SilkS")
+  (gr_text "VIDEO_IN" (at 112.5 51.87) (layer "F.SilkS")
     (effects (font (size 1.5 1.5) (thickness 0.25)))
   )
-  (gr_text "VIDEO_OUT" (at 186.7 53.1) (layer "F.SilkS")
+  (gr_text "VIDEO_OUT" (at 186.69 52.28) (layer "F.SilkS")
     (effects (font (size 1.5 1.5) (thickness 0.25)))
   )
-  (gr_text "VIDEO_RETURN" (at 184.25 147.35) (layer "F.SilkS")
+  (gr_text "VIDEO_RETURN" (at 184.62 148.15) (layer "F.SilkS")
     (effects (font (size 1.5 1.5) (thickness 0.25)))
   )
@@
     (effects (font (size 3 3) (thickness 0.4)))
   )
-  (gr_text "VIDEO_SEND" (at 114.55 147.55) (layer "F.SilkS")
+  (gr_text "VIDEO_SEND" (at 114.36 148.52) (layer "F.SilkS")
     (effects (font (size 1.5 1.5) (thickness 0.25)))
   )
